File: PCB/SARA.brd (EAGLE design)
At the start: 76.2 x 76.2 mm, 46 parts, among them U1 MAX9110EKA+T, U2 MAX9110EKA+T, U3 MAX9111EKA+T, U4 MAX9111EKA+T, U5 R-78B3.3-2.0, U6 R-78B3.3-2.0

Commit message: Finished Proto 1 PCB from cameron
Parts:
- removed JP1, JP2: (no value), pinhead:1X01
- added J1: 1935161, Screw Block:PHOENIX_1935161
- added J2: PJ-002AH, PJ-002AH:CUI_PJ-002AH
- L1: value 10uF -> 10uH
- moved C17 112.8 mm to (22.1, 48.1), turned to 180 degrees
- moved C16 112.8 mm to (22.1, 50.2), turned to 180 degrees
- moved C15 102.4 mm to (6.86, 43.0)
- moved C9 97.9 mm to (24.1, 66.1)
- moved C14 95.9 mm to (6.73, 40.7)
- moved C11 80.8 mm to (6.73, 38.6)
- moved C8 79.5 mm to (22.1, 52.1)
- moved C10 74.2 mm to (6.73, 36.2)
- moved C13 72.2 mm to (15.2, 22.4)
- moved C12 70.2 mm to (15.4, 24.8)
- moved C1 57.1 mm to (38.1, 61.1), turned to 180 degrees
- moved C2 53.6 mm to (38.1, 58.7)
- moved C7 47.9 mm to (42.9, 20.7), turned to 90 degrees
- moved C6 42.2 mm to (43.0, 31.9)
- moved C3 35.3 mm to (41.4, 55.4)
Connections:
- net GND: now also J1.2, J2.2, J2.3; no longer JP2.1
- net N$22: now also J1.1, J2.1; no longer JP1.1
Routing:
- net +3V3: track 123.8 -> 338.4 mm, vias 0 -> 8
- net I2C_SCL: track 27.1 -> 103.0 mm, vias 0 -> 2
- net I2C_SDA: track 29.3 -> 102.6 mm, vias 0 -> 3
- net GND: track 12.9 -> 68.7 mm, vias 2 -> 30
- net TX_DISABL_B: track 0.00 -> 32.0 mm
- net N$22: track 10.4 -> 27.7 mm
- net N$4: track 0.00 -> 2.83 mm
- net N$2: track 137.9 -> 139.2 mm, vias 2 -> 0
- net TX_DISABLE_A: track 29.0 -> 29.7 mm

Commit message: Added Tim's PCB v2 files
Parts:
- removed SFP_DOWNSTREAM, SFP_UPSTREAM: ZSFP+, zSFP+:ZSFP+
- added P1, P2: 74441-0010, 74441-0010:MOLEX_74441-0010
Connections:
- new net N$3: P1.6
- new net N$5: P1.7
- new net N$6: P1.9
- net +3V3: now also P1.15, P1.16, P2.15, P2.16; no longer SFP_DOWNSTREAM.15, SFP_DOWNSTREAM.16, SFP_UPSTREAM.15, SFP_UPSTREAM.16
- net GND: now also P1.1, P1.10, P1.11, P1.14, P1.17, P1.20, P2.1, P2.11, P2.14, P2.17, P2.20; no longer SFP_DOWNSTREAM.1, SFP_DOWNSTREAM.10, SFP_DOWNSTREAM.11, SFP_DOWNSTREAM.14, SFP_DOWNSTREAM.17, SFP_DOWNSTREAM.20, SFP_UPSTREAM.1, SFP_UPSTREAM.11, SFP_UPSTREAM.14, SFP_UPSTREAM.17, SFP_UPSTREAM.20
- net I2C_SCL: now also P1.5, P2.5; no longer SFP_DOWNSTREAM.5, SFP_UPSTREAM.5
- net I2C_SDA: now also P1.4, P2.4; no longer SFP_DOWNSTREAM.4, SFP_UPSTREAM.4
- net N$1: now also P2.8; no longer SFP_UPSTREAM.8
- net N$19: now also P1.8; no longer SFP_DOWNSTREAM.8
- net N$20: now also P1.2; no longer SFP_DOWNSTREAM.2
- net N$21: now also P2.2; no longer SFP_UPSTREAM.2
- net N$7: now also P2.10; no longer SFP_UPSTREAM.10
- net RXD_N: now also P2.12; no longer SFP_UPSTREAM.12
- net RXD_P: now also P2.13; no longer SFP_UPSTREAM.13
- net RXL_N: now also P1.12; no longer SFP_DOWNSTREAM.12
- net RXL_P: now also P1.13; no longer SFP_DOWNSTREAM.13
- net TXD_N: now also P2.19; no longer SFP_UPSTREAM.19
- net TXD_P: now also P2.18; no longer SFP_UPSTREAM.18
- net TXL_N: now also P1.19; no longer SFP_DOWNSTREAM.19
- net TXL_P: now also P1.18; no longer SFP_DOWNSTREAM.18
- net TX_DISABLE_A: now also P1.3; no longer SFP_DOWNSTREAM.3
- net TX_DISABL_B: now also P2.3; no longer SFP_UPSTREAM.3
Routing:
- net I2C_SDA: track 102.6 -> 72.1 mm
- net I2C_SCL: track 103.0 -> 74.2 mm
- net GND: track 68.7 -> 43.1 mm, vias 30 -> 21
- net +3V3: track 338.4 -> 329.9 mm
- net TXD_P: track 19.4 -> 14.8 mm
- net TXD_N: track 18.6 -> 14.4 mm
- net N$1: track 7.00 -> 4.65 mm
- net N$19: track 18.8 -> 17.3 mm
- net N$21: track 7.75 -> 6.27 mm
- net TXL_N: track 6.68 -> 5.38 mm
- net RXL_P: track 11.2 -> 9.95 mm
- net RXD_N: track 9.23 -> 7.96 mm
- net TX_DISABLE_A: track 29.7 -> 28.5 mm
- net N$20: track 23.4 -> 22.2 mm
- net TXL_P: track 7.37 -> 6.37 mm
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