File: PCB/SARA.sch (EAGLE design)
At the start: 46 parts, among them U1 MAX9110EKA+T, U2 MAX9110EKA+T, U3 MAX9111EKA+T, U4 MAX9111EKA+T, U5 R-78B3.3-2.0, U6 R-78B3.3-2.0

Commit message: 90% done routing, renamed stuff and added differental traces.
Parts:
- renumbered U$3 to SFP_DOWNSTREAM, U$4 to SFP_UPSTREAM
Connections:
- net N$6 renamed CLOCK
- removed net +3V1: C9.2, U1.VCC
- removed net +3V2: C10.2, C11.2, C12.2, C13.2, C14.2, C15.2, C16.2, C17.2, R4.1, R5.1, R6.1, R7.1, SFP_DOWNSTREAM.VCCR, SFP_DOWNSTREAM.VCCT, SFP_UPSTREAM.VCCR, SFP_UPSTREAM.VCCT
- net +3V3: now also C10.2, C11.2, C12.2, C13.2, C14.2, C15.2, C16.2, C17.2, C9.2, R4.1, R5.1, R6.1, R7.1, SFP_DOWNSTREAM.VCCR, SFP_DOWNSTREAM.VCCT, SFP_UPSTREAM.VCCR, SFP_UPSTREAM.VCCT, U1.VCC
Other:
- moved on the sheet: C12, C13, C16, C17

Commit message: Finished Proto 1 PCB from cameron
Parts:
- removed JP1, JP2: (no value), pinhead:PINHD-1X1
- added J1: 1935161, Screw Block:1935161
- added J2: PJ-002AH, PJ-002AH:PJ-002AH
- L1: value 10uF -> 10uH
Connections:
- net GND: now also J1.2, J2.2, J2.3; no longer JP2.1
- net N$22: now also J1.1, J2.1; no longer JP1.1
Other:
- note removed: "Molex Power Conn"
Changed lines of the file:
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@@
 <part name="SUPPLY20" library="supply2" library_urn="urn:adsk.eagle:library:372" deviceset="GND" device=""/>
 <part name="SUPPLY21" library="supply2" library_urn="urn:adsk.eagle:library:372" deviceset="GND" device=""/>
-<part name="JP1" library="pinhead" library_urn="urn:adsk.eagle:library:325" deviceset="PINHD-1X1" device="" package3d_urn="urn:adsk.eagle:package:22485/2"/>
-<part name="JP2" library="pinhead" library_urn="urn:adsk.eagle:library:325" deviceset="PINHD-1X1" device="" package3d_urn="urn:adsk.eagle:package:22485/2"/>
 <part name="SUPPLY22" library="supply2" library_urn="urn:adsk.eagle:library:372" deviceset="GND" device=""/>
 <part name="SFP_DOWNSTREAM" library="zSFP+" deviceset="ZSFP+" device=""/>
@@
 <part name="C17" library="capsmd" deviceset="C0603" device="" value="100nF"/>
 <part name="SUPPLY39" library="supply2" library_urn="urn:adsk.eagle:library:372" deviceset="GND" device=""/>
-<part name="L1" library="inductor-neosid" library_urn="urn:adsk.eagle:library:241" deviceset="MS50" device="" package3d_urn="urn:adsk.eagle:package:14699/1" value="10uF"/>
+<part name="L1" library="inductor-neosid" library_urn="urn:adsk.eagle:library:241" deviceset="MS50" device="" package3d_urn="urn:adsk.eagle:package:14699/1" value="10uH"/>
+<part name="J1" library="Screw Block" deviceset="1935161" device=""/>
+<part name="J2" library="PJ-002AH" deviceset="PJ-002AH" device=""/>
+<part name="SUPPLY40" library="supply2" library_urn="urn:adsk.eagle:library:372" deviceset="GND" device=""/>
 </parts>
 <sheets>
@@
 <plain>
 <text x="116.84" y="86.36" size="1.778" layer="91">JP3 is middle of board</text>
-<rectangle x1="-182.88" y1="162.56" x2="-154.94" y2="200.66" layer="91"/>
-<text x="-177.8" y="180.34" size="1.778" layer="91">Molex Power Conn</text>
-<text x="-177.8" y="180.34" size="1.778" layer="91">Molex Power Conn</text>
-<text x="-177.8" y="203.2" size="1.778" layer="91">Molex Power Conn</text>
 <text x="182.88" y="2.54" size="1.778" layer="91">EXT1 MCU</text>
 </plain>
@@
 <attribute name="VALUE" x="127.635" y="260.985" size="1.778" layer="96"/>
 </instance>
-<instance part="JP1" gate="G$1" x="-144.78" y="193.04" smashed="yes" rot="R180">
-<attribute name="NAME" x="-138.43" y="189.865" size="1.778" layer="95" rot="R180"/>
-<attribute name="VALUE" x="-138.43" y="198.12" size="1.778" layer="96" rot="R180"/>
-</instance>
-<instance part="JP2" gate="G$1" x="-139.7" y="165.1" smashed="yes">
-<attribute name="NAME" x="-146.05" y="168.275" size="1.778" layer="95"/>
-<attribute name="VALUE" x="-146.05" y="160.02" size="1.778" layer="96"/>
-</instance>
-<instance part="SUPPLY22" gate="GND" x="-142.24" y="162.56" smashed="yes">
-<attribute name="VALUE" x="-144.145" y="159.385" size="1.778" layer="96"/>
+<instance part="SUPPLY22" gate="GND" x="-147.32" y="208.28" smashed="yes">
+<attribute name="VALUE" x="-149.225" y="205.105" size="1.778" layer="96"/>
 </instance>
 <instance part="SFP_DOWNSTREAM" gate="G$1" x="7.62" y="289.56" smashed="yes"/>
@@
 <attribute name="NAME" x="-115.57" y="194.818" size="1.778" layer="95"/>
 <attribute name="VALUE" x="-115.57" y="189.484" size="1.778" layer="96"/>
+</instance>
+<instance part="J1" gate="G$1" x="-119.38" y="215.9" smashed="yes">
+<attribute name="NAME" x="-121.92548125" y="221.627340625" size="1.272740625" layer="95"/>
+<attribute name="VALUE" x="-121.92808125" y="208.25576875" size="1.274040625" layer="96"/>
+</instance>
+<instance part="J2" gate="G$1" x="-152.4" y="218.44" smashed="yes">
+<attribute name="NAME" x="-160.02723125" y="223.52481875" size="1.779690625" layer="95"/>
+<attribute name="VALUE" x="-160.031259375" y="213.3525" size="1.78063125" layer="96"/>
+</instance>
+<instance part="SUPPLY40" gate="GND" x="-134.62" y="210.82" smashed="yes">
+<attribute name="VALUE" x="-136.525" y="207.645" size="1.778" layer="96"/>
 </instance>
 </instances>
@@
 </segment>
 <segment>
-<pinref part="SUPPLY22" gate="GND" pin="GND"/>
-<pinref part="JP2" gate="G$1" pin="1"/>
-</segment>
-<segment>
 <pinref part="SUPPLY23" gate="GND" pin="GND"/>
 <pinref part="SFP_DOWNSTREAM" gate="G$1" pin="GND_5"/>
@@
 <pinref part="SUPPLY39" gate="GND" pin="GND"/>
 <pinref part="C17" gate="G$1" pin="1"/>
+</segment>
+<segment>
+<pinref part="J2" gate="G$1" pin="3"/>
+<pinref part="J2" gate="G$1" pin="2"/>
+<wire x1="-147.32" y1="218.44" x2="-147.32" y2="215.9" width="0.1524" layer="91"/>
+<pinref part="SUPPLY22" gate="GND" pin="GND"/>
+<wire x1="-147.32" y1="210.82" x2="-147.32" y2="215.9" width="0.1524" layer="91"/>
+<junction x="-147.32" y="215.9"/>
+</segment>
+<segment>
+<pinref part="J1" gate="G$1" pin="2"/>
+<pinref part="SUPPLY40" gate="GND" pin="GND"/>
+<wire x1="-127" y1="213.36" x2="-134.62" y2="213.36" width="0.1524" layer="91"/>
 </segment>
 </net>
@@
 <net name="N$22" class="0">
 <segment>
-<pinref part="JP1" gate="G$1" pin="1"/>
 <wire x1="-142.24" y1="193.04" x2="-121.92" y2="193.04" width="0.1524" layer="91"/>
 <pinref part="C4" gate="G$1" pin="2"/>
@@
 <junction x="-121.92" y="193.04"/>
 <pinref part="L1" gate="G$1" pin="1"/>
+<pinref part="J2" gate="G$1" pin="1"/>
+<wire x1="-147.32" y1="220.98" x2="-142.24" y2="220.98" width="0.1524" layer="91"/>
+<wire x1="-142.24" y1="220.98" x2="-142.24" y2="218.44" width="0.1524" layer="91"/>
+<pinref part="J1" gate="G$1" pin="1"/>
+<wire x1="-142.24" y1="218.44" x2="-142.24" y2="193.04" width="0.1524" layer="91"/>
+<wire x1="-127" y1="218.44" x2="-142.24" y2="218.44" width="0.1524" layer="91"/>
+<junction x="-142.24" y="218.44"/>
 </segment>
 </net>
@@
 </sheet>
 </sheets>
+<errors>
+</errors>
 </schematic>
 </drawing>

Commit message: Added Tim's PCB v2 files
Parts:
- removed SFP_DOWNSTREAM, SFP_UPSTREAM: ZSFP+, zSFP+:ZSFP+
- added P1, P2: 74441-0010, 74441-0010:74441-0010
Connections:
- new net N$3: P1.6
- new net N$5: P1.7
- new net N$6: P1.9
- net +3V3: now also P1.15, P1.16, P2.15, P2.16; no longer SFP_DOWNSTREAM.VCCR, SFP_DOWNSTREAM.VCCT, SFP_UPSTREAM.VCCR, SFP_UPSTREAM.VCCT
- net GND: now also P1.1, P1.10, P1.11, P1.14, P1.17, P1.20, P2.1, P2.11, P2.14, P2.17, P2.20; no longer SFP_DOWNSTREAM.GND_1, SFP_DOWNSTREAM.GND_2, SFP_DOWNSTREAM.GND_3, SFP_DOWNSTREAM.GND_4, SFP_DOWNSTREAM.GND_5, SFP_DOWNSTREAM.GND_6, SFP_UPSTREAM.GND_1, SFP_UPSTREAM.GND_3, SFP_UPSTREAM.GND_4, SFP_UPSTREAM.GND_5, SFP_UPSTREAM.GND_6
- net I2C_SCL: now also P1.5, P2.5; no longer SFP_DOWNSTREAM.SCL, SFP_UPSTREAM.SCL
- net I2C_SDA: now also P1.4, P2.4; no longer SFP_DOWNSTREAM.SDA, SFP_UPSTREAM.SDA
- net N$1: now also P2.8; no longer SFP_UPSTREAM.RX_LOS
- net N$19: now also P1.8; no longer SFP_DOWNSTREAM.RX_LOS
- net N$20: now also P1.2; no longer SFP_DOWNSTREAM.TX_FAULT
- net N$21: now also P2.2; no longer SFP_UPSTREAM.TX_FAULT
- net N$7: now also P2.10; no longer SFP_UPSTREAM.GND_2
- net RXD_N: now also P2.12; no longer SFP_UPSTREAM.RD-
- net RXD_P: now also P2.13; no longer SFP_UPSTREAM.RD+
- net RXL_N: now also P1.12; no longer SFP_DOWNSTREAM.RD-
- net RXL_P: now also P1.13; no longer SFP_DOWNSTREAM.RD+
- net TXD_N: now also P2.19; no longer SFP_UPSTREAM.TD-
- net TXD_P: now also P2.18; no longer SFP_UPSTREAM.TD+
- net TXL_N: now also P1.19; no longer SFP_DOWNSTREAM.TD-
- net TXL_P: now also P1.18; no longer SFP_DOWNSTREAM.TD+
- net TX_DISABLE_A: now also P1.3; no longer SFP_DOWNSTREAM.TX_DISABLE
- net TX_DISABL_B: now also P2.3; no longer SFP_UPSTREAM.TX_DISABLE
